Commit message: changed urdf

File: urdf/turtlebot3_waffle_pi_physical.urdf.xacro (robot description, xacro)
@@ -241,5 +241,5 @@
   <joint name="camera_joint" type="fixed">
 <!--	<origin xyz="0.073 -0.011 0.084" rpy="0 0.349 0"/> -->
-<origin xyz="0.073 -0.011 0.084" rpy="0 0.157 0"/>
+<origin xyz="0.073 -0.011 0.084" rpy="0 0 0"/>
     <parent link="base_link"/>
     <child link="camera_link"/>
